Commit message: Ultimo

File: src/rcauto_sim_pkg/urdf/rc_car.urdf.xacro (robot description, xacro)
@@ -48,4 +48,20 @@
   <xacro:property name="max_wheel_angular_velocity" value="${max_velocity / wheel_radius}"/>
   <xacro:property name="lidar_offsetX" value="${body_length/2 - wheel_radius}"/>
+  <!-- Physical Material Macros -->
+    <material name="Red">
+    	<color rgba="1.0 0 0 1.0"/>
+    </material>
+    <material name="Green">
+    	<color rgba="0 1.0 0 1.0"/>
+    </material>
+    <material name="Blue">
+    	<color rgba="0 0 1.0 0.5"/>
+    </material>
+    <material name="Black">
+    	<color rgba="0 0 0 1.0"/>
+    </material>
+    <material name="Aqua">
+    	<color rgba="0 1.0 1.0 1.0"/>
+    </material>
   <!-- Links -->
   <!-- Body Link -->
@@ -56,7 +72,5 @@
         <box size="${body_length} ${body_width} ${body_height}"/>
       </geometry>
-      <material name="body_material">
-        <color rgba="0.25 0.25 0.25 1.0"/>
-      </material>
+      <material name="Red"/>
     </visual>
     <collision>
@@ -67,4 +81,7 @@
     </collision>
   </link>
+  <gazebo reference="body_link">
+    <material>Gazebo/Red</material>
+  </gazebo>
   <!-- Body Base-->
   <link name="body_base_link">
@@ -74,7 +91,5 @@
         <box size="${body_length} ${body_width} ${body_height}"/>
       </geometry>
-      <material name="body_material">
-        <color rgba="0.25 0.25 0.25 1.0"/>
-      </material>
+      <material name="Red"/>
     </visual>
     <collision>
@@ -90,4 +105,7 @@
     </inertial>
   </link>
+  <gazebo reference="body_base_link">
+    <material>Gazebo/Red</material>
+  </gazebo>
   <!-- Front Left Wheel -->
   <link name="front_left_wheel_link">
@@ -97,7 +115,5 @@
         <cylinder radius="${wheel_radius}" length="${wheel_width}"/>
       </geometry>
-      <material name="wheel_material">
-        <color rgba="0.0 0.0 0.0 1.0"/>
-      </material>
+      <material name="Black"/>
     </visual>
     <collision>
@@ -113,4 +129,7 @@
     </inertial>
   </link>
+  <gazebo reference="front_left_wheel_link">
+    <material>Gazebo/Black</material>
+  </gazebo>
     <!-- Front Left Wheel Steering -->
   <link name="front_left_steering_link">
@@ -120,7 +139,5 @@
         <cylinder length="0.001" radius="0.01"/>
       </geometry>
-      <material name="wheel_material">
-        <color rgba="0.0 0.0 0.0 1.0"/>
-      </material>
+      <material name="Black"/>
     </visual>
     <collision>
@@ -136,4 +153,7 @@
     </inertial>
   </link>
+  <gazebo reference="front_left_steering_link">
+    <material>Gazebo/Black</material>
+  </gazebo>
   <!-- Front Right Wheel -->
   <link name="front_right_wheel_link">
@@ -143,7 +163,5 @@
         <cylinder radius="${wheel_radius}" length="${wheel_width}"/>
       </geometry>
-      <material name="wheel_material">
-        <color rgba="0.0 0.0 0.0 1.0"/>
-      </material>
+      <material name="Black"/>
     </visual>
     <collision>
@@ -159,4 +177,7 @@
     </inertial>
   </link>
+  <gazebo reference="front_right_wheel_link">
+    <material>Gazebo/Black</material>
+  </gazebo>
   <!-- Front Right Wheel Steering -->
   <link name="front_right_steering_link">
@@ -166,7 +187,5 @@
         <cylinder length="0.001" radius="0.01"/>
       </geometry>
-      <material name="wheel_material">
-        <color rgba="0.0 0.0 0.0 1.0"/>
-      </material>
+      <material name="Black"/>
     </visual>
     <collision>
@@ -182,4 +201,7 @@
     </inertial>
   </link>
+  <gazebo reference="front_right_steering_link">
+    <material>Gazebo/Black</material>
+  </gazebo>
   <!-- Rear Left Wheel -->
   <link name="rear_left_wheel_link">
@@ -189,7 +211,5 @@
         <cylinder radius="${wheel_radius}" length="${wheel_width}"/>
       </geometry>
-      <material name="wheel_material">
-        <color rgba="0.0 0.0 0.0 1.0"/>
-      </material>
+      <material name="Black"/>
     </visual>
     <collision>
@@ -205,4 +225,7 @@
     </inertial>
   </link>
+  <gazebo reference="rear_left_wheel_link">
+    <material>Gazebo/Black</material>
+  </gazebo>
   <!-- Rear Right Wheel -->
   <link name="rear_right_wheel_link">
@@ -212,7 +235,5 @@
         <cylinder radius="${wheel_radius}" length="${wheel_width}"/>
       </geometry>
-      <material name="wheel_material">
-        <color rgba="0.0 0.0 0.0 1.0"/>
-      </material>
+      <material name="Black"/>
     </visual>
     <collision>
@@ -228,4 +249,7 @@
     </inertial>
   </link>
+  <gazebo reference="rear_right_wheel_link">
+    <material>Gazebo/Black</material>
+  </gazebo>
   <!-- Joints -->
   <!-- Body Base Joint -->

File: src/rcauto_sim_pkg/urdf/spechCar.urdf.xacro (robot description, xacro)
@@ -48,4 +48,20 @@
   <xacro:property name="max_wheel_angular_velocity" value="${max_velocity / wheel_radius}"/>
   <xacro:property name="lidar_offsetX" value="${body_length/2 - wheel_radius}"/>
+  <!-- Physical Material Macros -->
+    <material name="Red">
+    	<color rgba="1.0 0 0 1.0"/>
+    </material>
+    <material name="Green">
+    	<color rgba="0 1.0 0 1.0"/>
+    </material>
+    <material name="Blue">
+    	<color rgba="0 0 1.0 0.5"/>
+    </material>
+    <material name="Black">
+    	<color rgba="0 0 0 1.0"/>
+    </material>
+    <material name="Aqua">
+    	<color rgba="0 1.0 1.0 1.0"/>
+    </material>
   <!-- Links -->
   <!-- Body Link -->
@@ -56,7 +72,5 @@
         <box size="${body_length} ${body_width} ${body_height}"/>
       </geometry>
-      <material name="body_material">
-        <color rgba="0.25 0.25 0.25 1.0"/>
-      </material>
+      <material name="Red"/>
     </visual>
     <collision>
@@ -67,4 +81,7 @@
     </collision>
   </link>
+  <gazebo reference="body_link">
+    <material>Gazebo/Red</material>
+  </gazebo>
   <!-- Body Base-->
   <link name="body_base_link">
@@ -74,7 +91,5 @@
         <box size="${body_length} ${body_width} ${body_height}"/>
       </geometry>
-      <material name="body_material">
-        <color rgba="0.25 0.25 0.25 1.0"/>
-      </material>
+      <material name="Red"/>
     </visual>
     <collision>
@@ -90,4 +105,7 @@
     </inertial>
   </link>
+  <gazebo reference="body_base_link">
+    <material>Gazebo/Red</material>
+  </gazebo>
   <!-- Front Left Wheel -->
   <link name="front_left_wheel_link">
@@ -97,7 +115,5 @@
         <cylinder radius="${wheel_radius}" length="${wheel_width}"/>
       </geometry>
-      <material name="wheel_material">
-        <color rgba="0.0 0.0 0.0 1.0"/>
-      </material>
+      <material name="Black"/>
     </visual>
     <collision>
@@ -113,4 +129,7 @@
     </inertial>
   </link>
+  <gazebo reference="front_left_wheel_link">
+    <material>Gazebo/Black</material>
+  </gazebo>
     <!-- Front Left Wheel Steering -->
   <link name="front_left_steering_link">
@@ -120,7 +139,5 @@
         <cylinder length="0.001" radius="0.01"/>
       </geometry>
-      <material name="wheel_material">
-        <color rgba="0.0 0.0 0.0 1.0"/>
-      </material>
+      <material name="Black"/>
     </visual>
     <collision>
@@ -136,4 +153,7 @@
     </inertial>
   </link>
+  <gazebo reference="front_left_steering_link">
+    <material>Gazebo/Black</material>
+  </gazebo>
   <!-- Front Right Wheel -->
   <link name="front_right_wheel_link">
@@ -143,7 +163,5 @@
         <cylinder radius="${wheel_radius}" length="${wheel_width}"/>
       </geometry>
-      <material name="wheel_material">
-        <color rgba="0.0 0.0 0.0 1.0"/>
-      </material>
+      <material name="Black"/>
     </visual>
     <collision>
@@ -159,4 +177,7 @@
     </inertial>
   </link>
+  <gazebo reference="front_right_wheel_link">
+    <material>Gazebo/Black</material>
+  </gazebo>
   <!-- Front Right Wheel Steering -->
   <link name="front_right_steering_link">
@@ -166,7 +187,5 @@
         <cylinder length="0.001" radius="0.01"/>
       </geometry>
-      <material name="wheel_material">
-        <color rgba="0.0 0.0 0.0 1.0"/>
-      </material>
+      <material name="Black"/>
     </visual>
     <collision>
@@ -182,4 +201,7 @@
     </inertial>
   </link>
+  <gazebo reference="front_right_steering_link">
+    <material>Gazebo/Black</material>
+  </gazebo>
   <!-- Rear Left Wheel -->
   <link name="rear_left_wheel_link">
@@ -189,7 +211,5 @@
         <cylinder radius="${wheel_radius}" length="${wheel_width}"/>
       </geometry>
-      <material name="wheel_material">
-        <color rgba="0.0 0.0 0.0 1.0"/>
-      </material>
+      <material name="Black"/>
     </visual>
     <collision>
@@ -205,4 +225,7 @@
     </inertial>
   </link>
+  <gazebo reference="rear_left_wheel_link">
+    <material>Gazebo/Black</material>
+  </gazebo>
   <!-- Rear Right Wheel -->
   <link name="rear_right_wheel_link">
@@ -212,7 +235,5 @@
         <cylinder radius="${wheel_radius}" length="${wheel_width}"/>
       </geometry>
-      <material name="wheel_material">
-        <color rgba="0.0 0.0 0.0 1.0"/>
-      </material>
+      <material name="Black"/>
     </visual>
     <collision>
@@ -228,4 +249,7 @@
     </inertial>
   </link>
+  <gazebo reference="rear_right_wheel_link">
+    <material>Gazebo/Black</material>
+  </gazebo>
   <!-- Joints -->
   <!-- Body Base Joint -->
@@ -355,7 +379,5 @@
         <cylinder radius="0.1" length="0.2"/>
       </geometry>
-      <material name="yellow">
-        <color rgba="1 1 0 1"/>
-      </material>
+      <material name="Blue"/>
     </visual>
     <collision name="lidar_collision">
@@ -365,4 +387,7 @@
     </collision>
   </link>
+  <gazebo reference="lidar_link">
+    <material>Gazebo/Blue</material>
+  </gazebo>
   <!-- Junta fija para montar el LIDAR sobre el chasis -->
   <joint name="lidar_joint" type="fixed">
